Commit message: roboschool cpp api

File: roboschool/models_household/ball-small/ball.urdf (robot description, URDF)
Before this commit: robot ball, 1 links, 0 joints
Links:
- link body: geometry collision sphere radius=0.05; visual sphere radius=0.01

File: roboschool/models_household/ball/ball.urdf (robot description, URDF)
Before this commit: robot ball, 1 links, 0 joints
Links:
- link body: geometry collision sphere radius=0.04; visual mesh filename=ball.obj
